Commit message: ready for rviz

File: src/kilin_description/urdf/kilin.urdf (robot description, URDF)
Before this commit: robot URDF, 17 links, 16 joints
Links:
- link FL_LowerLeg: geometry collision mesh filename=package://kilin_description/meshes/FL_LowerLeg.STL; visual mesh filename=package://kilin_description/meshes/FL_LowerLeg.STL
- link FL_Thigh: geometry collision mesh filename=package://kilin_description/meshes/FL_Thigh.STL; visual mesh filename=package://kilin_description/meshes/FL_Thigh.STL
- link FL_UpperLeg: geometry collision mesh filename=package://kilin_description/meshes/FL_UpperLeg.STL; visual mesh filename=package://kilin_description/meshes/FL_UpperLeg.STL
- link FL_Wheel: geometry collision mesh filename=package://kilin_description/meshes/FL_Wheel.STL; visual mesh filename=package://kilin_description/meshes/FL_Wheel.STL
- link FR_LowerLeg: geometry collision mesh filename=package://kilin_description/meshes/FR_LowerLeg.STL; visual mesh filename=package://kilin_description/meshes/FR_LowerLeg.STL
- link FR_Thigh: geometry collision mesh filename=package://kilin_description/meshes/FR_Thigh.STL; visual mesh filename=package://kilin_description/meshes/FR_Thigh.STL
- link FR_UpperLeg: geometry collision mesh filename=package://kilin_description/meshes/FR_UpperLeg.STL; visual mesh filename=package://kilin_description/meshes/FR_UpperLeg.STL
- link FR_Wheel: geometry collision mesh filename=package://kilin_description/meshes/FR_Wheel.STL; visual mesh filename=package://kilin_description/meshes/FR_Wheel.STL
- link RL_LowerLeg: geometry collision mesh filename=package://kilin_description/meshes/RL_LowerLeg.STL; visual mesh filename=package://kilin_description/meshes/RL_LowerLeg.STL
- link RL_Thigh: geometry collision mesh filename=package://kilin_description/meshes/RL_Thigh.STL; visual mesh filename=package://kilin_description/meshes/RL_Thigh.STL
- link RL_UpperLeg: geometry collision mesh filename=package://kilin_description/meshes/RL_UpperLeg.STL; visual mesh filename=package://kilin_description/meshes/RL_UpperLeg.STL
- link RL_Wheel: geometry collision mesh filename=package://kilin_description/meshes/RL_Wheel.STL; visual mesh filename=package://kilin_description/meshes/RL_Wheel.STL
- link RR_LowerLeg: geometry collision mesh filename=package://kilin_description/meshes/RR_LowerLeg.STL; visual mesh filename=package://kilin_description/meshes/RR_LowerLeg.STL
- link RR_Thigh: geometry collision mesh filename=package://kilin_description/meshes/RR_Thigh.STL; visual mesh filename=package://kilin_description/meshes/RR_Thigh.STL
- link RR_UpperLeg: geometry collision mesh filename=package://kilin_description/meshes/RR_UpperLeg.STL; visual mesh filename=package://kilin_description/meshes/RR_UpperLeg.STL
- link RR_Wheel: geometry collision mesh filename=package://kilin_description/meshes/RR_Wheel.STL; visual mesh filename=package://kilin_description/meshes/RR_Wheel.STL
- link base_link: geometry collision mesh filename=package://kilin_description/meshes/base_link.STL; visual mesh filename=package://kilin_description/meshes/base_link.STL
